Commit message: Update ballbot.urdf.xacro Reduced redundancy with xacro macros and properties.

File: ballbot_description/urdf/ballbot.urdf.xacro (robot description, xacro)
@@ -1,131 +1,156 @@
 <?xml version="1.0"?>
-<robot name="collector_bot">
-  <!-- =================================================================== -->
-  <!-- |                           MATERIALS                             | -->
-  <!-- =================================================================== -->
-  <material name="blue">
-    <color rgba="0.0 0.0 0.8 1.0"/>
-  </material>
-  <material name="black">
-    <color rgba="0.0 0.0 0.0 1.0"/>
-  </material>
-  <material name="grey">
-    <color rgba="0.5 0.5 0.5 1.0"/>
-  </material>
-  <material name="green">
-    <color rgba="0.0 0.8 0.0 1.0"/>
-  </material>
-  <material name="red">
-    <color rgba="0.8 0.0 0.0 1.0"/>
-  </material>
-  <!-- =================================================================== -->
-  <!-- |                            BASE LINK (CHASSIS)                  | -->
-  <!-- =================================================================== -->
+<robot xmlns:xacro="http://www.ros.org/wiki/xacro" name="collector_bot">
+  <xacro:property name="chassis_len" value="0.5"/>
+  <xacro:property name="chassis_width" value="0.5"/>
+  <xacro:property name="chassis_height" value="0.3"/>
+  <xacro:property name="chassis_mass" value="3.0"/>
+  <xacro:property name="chassis_z_offset" value="0.20"/>
+  <xacro:property name="wheel_radius" value="0.05"/>
+  <xacro:property name="wheel_width" value="0.04"/>
+  <xacro:property name="wheel_mass" value="0.5"/>
+  <xacro:property name="wheel_y_offset" value="0.27"/>
+  <xacro:property name="wheel_z_offset" value="0.05"/>
+  <xacro:property name="castor_radius" value="0.04"/>
+  <xacro:property name="castor_mass" value="0.2"/>
+  <xacro:property name="castor_x_offset" value="-0.2"/>
+  <xacro:property name="arm_len" value="0.6"/>
+  <xacro:property name="arm_width" value="0.05"/>
+  <xacro:property name="arm_height" value="0.3"/>
+  <xacro:property name="arm_mass" value="1.5"/>
+  <xacro:property name="arm_angle" value="0.523"/> <xacro:property name="flap_len" value="0.3"/>
+  <xacro:property name="flap_width" value="0.02"/>
+  <xacro:property name="flap_height" value="0.3"/>
+  <xacro:property name="flap_mass" value="0.3"/>
+  <material name="blue"><color rgba="0.0 0.0 0.8 1.0"/></material>
+  <material name="black"><color rgba="0.0 0.0 0.0 1.0"/></material>
+  <material name="grey"><color rgba="0.5 0.5 0.5 1.0"/></material>
+  <material name="green"><color rgba="0.0 0.8 0.0 1.0"/></material>
+  <material name="red"><color rgba="0.8 0.0 0.0 1.0"/></material>
+  <xacro:macro name="box_inertia" params="m x y z">
+    <inertial>
+      <mass value="${m}"/>
+      <inertia ixx="${m/12.0 * (y*y + z*z)}" ixy="0.0" ixz="0.0"
+               iyy="${m/12.0 * (x*x + z*z)}" iyz="0.0"
+               izz="${m/12.0 * (x*x + y*y)}"/>
+    </inertial>
+  </xacro:macro>
+  <xacro:macro name="cylinder_inertia" params="m r h">
+    <inertial>
+      <mass value="${m}"/>
+      <inertia ixx="${m/12.0 * (3*r*r + h*h)}" ixy="0.0" ixz="0.0"
+               iyy="${m/12.0 * (3*r*r + h*h)}" iyz="0.0"
+               izz="${m/2.0 * (r*r)}"/>
+    </inertial>
+  </xacro:macro>
+  <xacro:macro name="sphere_inertia" params="m r">
+    <inertial>
+      <mass value="${m}"/>
+      <inertia ixx="${2.0/5.0 * m * r*r}" ixy="0.0" ixz="0.0"
+               iyy="${2.0/5.0 * m * r*r}" iyz="0.0"
+               izz="${2.0/5.0 * m * r*r}"/>
+    </inertial>
+  </xacro:macro>
+  <xacro:macro name="drive_wheel" params="prefix reflect">
+    <link name="${prefix}_wheel">
+      <visual>
+        <origin xyz="0 0 0" rpy="${pi/2} 0 0"/>
+        <geometry>
+          <cylinder radius="${wheel_radius}" length="${wheel_width}"/>
+        </geometry>
+        <material name="black"/>
+      </visual>
+      <collision>
+        <origin xyz="0 0 0" rpy="${pi/2} 0 0"/>
+        <geometry>
+          <cylinder radius="${wheel_radius}" length="${wheel_width}"/>
+        </geometry>
+      </collision>
+      <xacro:cylinder_inertia m="${wheel_mass}" r="${wheel_radius}" h="${wheel_width}"/>
+    </link>
+    <joint name="${prefix}_wheel_joint" type="continuous">
+      <parent link="base_link"/>
+      <child link="${prefix}_wheel"/>
+      <origin xyz="0 ${reflect * wheel_y_offset} ${wheel_z_offset}" rpy="0 0 0"/>
+      <axis xyz="0 1 0"/>
+    </joint>
+  </xacro:macro>
+  <xacro:macro name="collector_arm" params="prefix reflect angle limit_lower limit_upper">
+    <link name="${prefix}_arm">
+      <visual>
+        <geometry>
+          <box size="${arm_len} ${arm_width} ${arm_height}"/>
+        </geometry>
+        <material name="green"/>
+      </visual>
+      <collision>
+        <geometry>
+          <box size="${arm_len} ${arm_width} ${arm_height}"/>
+        </geometry>
+      </collision>
+      <xacro:box_inertia m="${arm_mass}" x="${arm_len}" y="${arm_width}" z="${arm_height}"/>
+    </link>
+    <joint name="${prefix}_arm_joint" type="fixed">
+      <parent link="base_link"/>
+      <child link="${prefix}_arm"/>
+      <origin xyz="0.51 ${reflect * 0.40} ${chassis_z_offset}" rpy="0 0 ${reflect * angle}"/>
+    </joint>
+    <link name="${prefix}_flap">
+      <visual>
+        <origin xyz="${flap_len/2} 0 0" rpy="0 0 0"/>
+        <geometry>
+          <box size="${flap_len} ${flap_width} ${flap_height}"/>
+        </geometry>
+        <material name="red"/>
+      </visual>
+      <collision>
+        <origin xyz="${flap_len/2} 0 0" rpy="0 0 0"/>
+        <geometry>
+          <box size="${flap_len} ${flap_width} ${flap_height}"/>
+        </geometry>
+      </collision>
+      <inertial>
+        <origin xyz="${flap_len/2} 0 0" rpy="0 0 0"/>
+        <mass value="${flap_mass}"/>
+        <inertia ixx="${flap_mass/12.0 * (flap_width*flap_width + flap_height*flap_height)}" ixy="0.0" ixz="0.0"
+                 iyy="${flap_mass/12.0 * (flap_len*flap_len + flap_height*flap_height)}" iyz="0.0"
+                 izz="${flap_mass/12.0 * (flap_len*flap_len + flap_width*flap_width)}"/>
+      </inertial>
+    </link>
+    <joint name="${prefix}_flap_joint" type="revolute">
+      <parent link="${prefix}_arm"/>
+      <child link="${prefix}_flap"/>
+      <origin xyz="${arm_len/2} 0 0" rpy="0 0 0"/>
+      <axis xyz="0 0 1"/>
+      <limit lower="${limit_lower}" upper="${limit_upper}" effort="10.0" velocity="1.0"/>
+    </joint>
+  </xacro:macro>
   <link name="base_link">
     <visual>
-      <!--
-         New Height: 30cm (0.3).
-         Ground is Z=0. Wheel radius is 0.05. Chassis bottom sits at Z=0.05.
-         Center of chassis is Z = 0.05 + (0.3 / 2) = 0.20.
-      -->
-      <origin xyz="0 0 0.20" rpy="0 0 0"/>
-      <geometry>
-        <!-- 50cm wide (Y), 50cm long (X), 30cm tall (Z) -->
-        <box size="0.5 0.5 0.3"/>
+      <origin xyz="0 0 ${chassis_z_offset}" rpy="0 0 0"/>
+      <geometry>
+        <box size="${chassis_len} ${chassis_width} ${chassis_height}"/>
       </geometry>
       <material name="blue"/>
     </visual>
     <collision>
-      <origin xyz="0 0 0.20" rpy="0 0 0"/>
-      <geometry>
-        <box size="0.5 0.5 0.3"/>
-      </geometry>
-    </collision>
-    <inertial>
-      <origin xyz="0 0 0.20" rpy="0 0 0"/>
-      <!-- Mass reduced (approx 3kg) for smaller volume -->
-      <mass value="3.0"/>
-      <inertia
-        ixx="0.085" ixy="0.0" ixz="0.0"
-        iyy="0.085" iyz="0.0"
-        izz="0.125"/>
-    </inertial>
-  </link>
-  <!-- =================================================================== -->
-  <!-- |                         DRIVE WHEELS (LEFT & RIGHT)             | -->
-  <!-- =================================================================== -->
-  <!-- Left Wheel -->
-  <link name="left_wheel">
-    <visual>
-      <!-- Visuals are rotated 90 deg on X to align with the Y-axis joint -->
-      <origin xyz="0 0 0" rpy="1.5707 0 0" />
-      <geometry>
-        <!-- 10cm diameter, 4cm wide -->
-        <cylinder radius="0.05" length="0.04"/>
-      </geometry>
-      <material name="black"/>
-    </visual>
-    <collision>
-      <origin xyz="0 0 0" rpy="1.5707 0 0" />
-      <geometry>
-        <cylinder radius="0.05" length="0.04"/>
-      </geometry>
-    </collision>
-    <inertial>
-      <!-- Mass of 0.5kg for the wheel -->
-      <mass value="0.5"/>
-      <inertia
-        ixx="0.000378" ixy="0.0" ixz="0.0"
-        iyy="0.000378" iyz="0.0"
-        izz="0.000625"/>
-    </inertial>
-  </link>
-  <joint name="left_wheel_joint" type="continuous">
-    <parent link="base_link"/>
-    <child link="left_wheel"/>
-    <!-- Positioned just outside the 50cm chassis on the Y-axis -->
-    <!-- Z=0.05 places the axle 5cm above ground (0,0,0) -->
-    <origin xyz="0 0.27 0.05" rpy="0 0 0"/>
-    <!-- Spin axis is Y -->
-    <axis xyz="0 1 0"/>
-  </joint>
-  <!-- Right Wheel -->
-  <link name="right_wheel">
-    <visual>
-      <origin xyz="0 0 0" rpy="1.5707 0 0" />
-      <geometry>
-        <cylinder radius="0.05" length="0.04"/>
-      </geometry>
-      <material name="black"/>
-    </visual>
-    <collision>
-      <origin xyz="0 0 0" rpy="1.5707 0 0" />
-      <geometry>
-        <cylinder radius="0.05" length="0.04"/>
-      </geometry>
-    </collision>
-    <inertial>
-      <mass value="0.5"/>
-      <inertia
-        ixx="0.000378" ixy="0.0" ixz="0.0"
-        iyy="0.000378" iyz="0.0"
-        izz="0.000625"/>
-    </inertial>
-  </link>
-  <joint name="right_wheel_joint" type="continuous">
-    <parent link="base_link"/>
-    <child link="right_wheel"/>
-    <!-- Z=0.05 places the axle 5cm above ground (0,0,0) -->
-    <origin xyz="0 -0.27 0.05" rpy="0 0 0"/>
-    <axis xyz="0 1 0"/>
-  </joint>
-  <!-- =================================================================== -->
-  <!-- |                           CASTOR WHEEL                          | -->
-  <!-- =================================================================== -->
+      <origin xyz="0 0 ${chassis_z_offset}" rpy="0 0 0"/>
+      <geometry>
+        <box size="${chassis_len} ${chassis_width} ${chassis_height}"/>
+      </geometry>
+    </collision>
+    <inertial>
+        <origin xyz="0 0 ${chassis_z_offset}" rpy="0 0 0"/>
+        <mass value="${chassis_mass}"/>
+        <inertia ixx="${chassis_mass/12.0 * (chassis_width*chassis_width + chassis_height*chassis_height)}" ixy="0.0" ixz="0.0"
+                 iyy="${chassis_mass/12.0 * (chassis_len*chassis_len + chassis_height*chassis_height)}" iyz="0.0"
+                 izz="${chassis_mass/12.0 * (chassis_len*chassis_len + chassis_width*chassis_width)}"/>
+    </inertial>
+  </link>
+  <xacro:drive_wheel prefix="left" reflect="1"/>
+  <xacro:drive_wheel prefix="right" reflect="-1"/>
   <link name="castor_wheel">
     <visual>
       <geometry>
-        <!-- 8cm diameter sphere -->
-        <sphere radius="0.04"/>
+        <sphere radius="${castor_radius}"/>
       </geometry>
       <material name="grey"/>
@@ -133,33 +158,17 @@
     <collision>
       <geometry>
-        <sphere radius="0.04"/>
-      </geometry>
-    </collision>
-    <inertial>
-      <!-- Mass of 0.2kg -->
-      <mass value="0.2"/>
-      <inertia
-        ixx="0.000128" ixy="0.0" ixz="0.0"
-        iyy="0.000128" iyz="0.0"
-        izz="0.000128"/>
-    </inertial>
+        <sphere radius="${castor_radius}"/>
+      </geometry>
+    </collision>
+    <xacro:sphere_inertia m="${castor_mass}" r="${castor_radius}"/>
   </link>
   <joint name="castor_wheel_joint" type="fixed">
     <parent link="base_link"/>
     <child link="castor_wheel"/>
-    <!--
-      Ground is Z=0.
-      Castor (r=0.04) center must be at Z=0.04 to touch ground.
-      Rear position: X = -0.2
-    -->
-    <origin xyz="-0.2 0 0.04" rpy="0 0 0"/>
+    <origin xyz="${castor_x_offset} 0 ${castor_radius}" rpy="0 0 0"/>
   </joint>
-  <!-- =================================================================== -->
-  <!-- |                       VERTICAL POLE & LIDAR                     | -->
-  <!-- =================================================================== -->
   <link name="vertical_pole">
     <visual>
       <geometry>
-        <!-- Shortened pole: 5cm tall, 4cm diameter -->
         <cylinder radius="0.02" length="0.05"/>
       </geometry>
@@ -171,25 +180,12 @@
       </geometry>
     </collision>
-    <inertial>
-      <!-- Mass reduced to 0.1kg -->
-      <mass value="0.1"/>
-      <inertia
-        ixx="0.00003" ixy="0.0" ixz="0.0"
-        iyy="0.00003" iyz="0.0"
-        izz="0.00002"/>
-    </inertial>
+    <xacro:cylinder_inertia m="0.1" r="0.02" h="0.05"/>
   </link>
   <joint name="vertical_pole_joint" type="fixed">
     <parent link="base_link"/>
     <child link="vertical_pole"/>
-    <!--
-      Attached to the center (X=0, Y=0).
-      Chassis bottom Z=0.05. Chassis height 0.3. Top is Z=0.35.
-      Pole center (0.05 / 2 = 0.025) is placed at Z = 0.35 + 0.025 = 0.375.
-    -->
     <origin xyz="0 0 0.375" rpy="0 0 0"/>
   </joint>
-  <!-- Lidar Link -->
-  <link name="lidar">
+  <link name="lidar_link">
     <visual>
       <geometry>
@@ -203,159 +199,12 @@
       </geometry>
     </collision>
-    <inertial>
-      <!-- Mass of 0.3kg -->
-      <mass value="0.3"/>
-      <inertia
-        ixx="0.00025" ixy="0.0" ixz="0.0"
-        iyy="0.00025" iyz="0.0"
-        izz="0.000375"/>
-    </inertial>
+    <xacro:cylinder_inertia m="0.3" r="0.05" h="0.05"/>
   </link>
   <joint name="lidar_joint" type="fixed">
     <parent link="vertical_pole"/>
-    <child link="lidar"/>
-    <!--
-      Placed on top of the short pole.
-      Pole's local top is at Z=0.025.
-      Lidar center (0.05 / 2 = 0.025) is placed at
-      Z = 0.025 + 0.025 = 0.05.
-    -->
+    <child link="lidar_link"/>
     <origin xyz="0 0 0.05" rpy="0 0 0"/>
   </joint>
-  <!-- =================================================================== -->
-  <!-- |                       BALL COLLECTOR ARMS (V-SHAPE)             | -->
-  <!-- =================================================================== -->
-  <!--  -->
-  <!-- Left Arm -->
-  <link name="left_arm">
-    <visual>
-      <geometry>
-        <!-- 60cm long, 5cm wide, 30cm tall -->
-        <box size="0.6 0.05 0.3"/>
-      </geometry>
-      <material name="green"/>
-    </visual>
-    <collision>
-      <geometry>
-        <box size="0.6 0.05 0.3"/>
-      </geometry>
-    </collision>
-    <inertial>
-      <!-- Mass reduced to 1.5kg -->
-      <mass value="1.5"/>
-      <inertia
-        ixx="0.0115" ixy="0.0" ixz="0.0"
-        iyy="0.0562" iyz="0.0"
-        izz="0.0453"/>
-    </inertial>
-  </link>
-  <joint name="left_arm_joint" type="fixed">
-    <parent link="base_link"/>
-    <child link="left_arm"/>
-    <!--
-      Attached to the front-left.
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
Commit message: Created ballbot_control
TODO: Get this to work...
EOD: launched empty world, polished xacro, and began ballbot control work.

File: ballbot_description/urdf/ballbot.urdf.xacro (robot description, xacro)
@@ -1,4 +1,4 @@
 <?xml version="1.0"?>
-<robot xmlns:xacro="http://www.ros.org/wiki/xacro" name="collector_bot">
+<robot xmlns:xacro="http://www.ros.org/wiki/xacro" name="ballbot">
   <xacro:property name="chassis_len" value="0.5"/>
   <xacro:property name="chassis_width" value="0.5"/>
@@ -18,5 +18,6 @@
   <xacro:property name="arm_height" value="0.3"/>
   <xacro:property name="arm_mass" value="1.5"/>
-  <xacro:property name="arm_angle" value="0.523"/> <xacro:property name="flap_len" value="0.3"/>
+  <xacro:property name="arm_angle" value="0.523"/>
+  <xacro:property name="flap_len" value="0.3"/>
   <xacro:property name="flap_width" value="0.02"/>
   <xacro:property name="flap_height" value="0.3"/>
@@ -208,7 +209,42 @@
   <xacro:collector_arm prefix="left" reflect="1" angle="${arm_angle}" limit_lower="-1.57" limit_upper="0.0"/>
   <xacro:collector_arm prefix="right" reflect="-1" angle="${arm_angle}" limit_lower="0.0" limit_upper="1.57"/>
+  <!-- ROS2 CONTROL -->
+  <ros2_control name="GazeboSimSystem" type="system">
+    <hardware>
+      <plugin>gz_ros2_control/GazeboSimSystem</plugin>
+    </hardware>
+    <!-- Wheels -->
+    <joint name="left_wheel_joint">
+      <command_interface name="velocity">
+        <param name="min">-10</param>
+        <param name="max">10</param>
+      </command_interface>
+      <state_interface name="velocity"/>
+      <state_interface name="position"/>
+    </joint>
+    <joint name="right_wheel_joint">
+      <command_interface name="velocity">
+        <param name="min">-10</param>
+        <param name="max">10</param>
+      </command_interface>
+      <state_interface name="velocity"/>
+      <state_interface name="position"/>
+    </joint>
+    <!-- Flaps -->
+    <joint name="left_flap_joint">
+      <command_interface name="position"/>
+      <state_interface name="position"/>
+      <state_interface name="velocity"/>
+    </joint>
+    <joint name="right_flap_joint">
+      <command_interface name="position"/>
+      <state_interface name="position"/>
+      <state_interface name="velocity"/>
+    </joint>
+  </ros2_control>
+  <!-- Gazebo Plugin for ros2_control -->
   <gazebo>
-    <plugin filename="gz-sim-joint-state-publisher-system"
-            name="gz::sim::systems::JointStatePublisher">
+    <plugin filename="gz_ros2_control-system" name="gz_ros2_control::GazeboSimROS2ControlPlugin">
+      <parameters>$(find ballbot_control)/config/ballbot_controllers.yaml</parameters>
     </plugin>
   </gazebo>

Commit message: WIP: ballbot_control ballbot_description

File: ballbot_description/urdf/ballbot.urdf.xacro (robot description, xacro)
@@ -74,4 +74,6 @@
       <origin xyz="0 ${reflect * wheel_y_offset} ${wheel_z_offset}" rpy="0 0 0"/>
       <axis xyz="0 1 0"/>
+      <!-- CRITICAL FIX: Limits are required for Gazebo to apply effort -->
+      <limit effort="50.0" velocity="20.0"/>
     </joint>
   </xacro:macro>
@@ -126,4 +128,11 @@
     </joint>
   </xacro:macro>
+  <!-- FIX: Added base_footprint to silence KDL warning about root link inertia -->
+  <link name="base_footprint"/>
+  <joint name="base_joint" type="fixed">
+    <parent link="base_footprint"/>
+    <child link="base_link"/>
+    <origin xyz="0 0 0" rpy="0 0 0"/>
+  </joint>
   <link name="base_link">
     <visual>

Commit message: Update ballbot_control, ballbot_launch, ballbot_description
Adjusted launch files to load gazebo empty world, rviz, and controllers
Adjusted urdf to connect differential drive controller to gazebo
Adjusted arm mass and castor wheel mass to pull back center of gravity and eliminate forward tilting.

TODO: Adjust flap controllers to work appropriately.

File: ballbot_description/urdf/ballbot.urdf.xacro (robot description, xacro)
@@ -12,15 +12,15 @@
   <xacro:property name="wheel_z_offset" value="0.05"/>
   <xacro:property name="castor_radius" value="0.04"/>
-  <xacro:property name="castor_mass" value="0.2"/>
+  <xacro:property name="castor_mass" value="1.5"/>
   <xacro:property name="castor_x_offset" value="-0.2"/>
   <xacro:property name="arm_len" value="0.6"/>
   <xacro:property name="arm_width" value="0.05"/>
   <xacro:property name="arm_height" value="0.3"/>
-  <xacro:property name="arm_mass" value="1.5"/>
+  <xacro:property name="arm_mass" value="0.04"/>
   <xacro:property name="arm_angle" value="0.523"/>
   <xacro:property name="flap_len" value="0.3"/>
   <xacro:property name="flap_width" value="0.02"/>
   <xacro:property name="flap_height" value="0.3"/>
-  <xacro:property name="flap_mass" value="0.3"/>
+  <xacro:property name="flap_mass" value="0.01"/>
   <material name="blue"><color rgba="0.0 0.0 0.8 1.0"/></material>
   <material name="black"><color rgba="0.0 0.0 0.0 1.0"/></material>
@@ -77,4 +77,10 @@
       <limit effort="50.0" velocity="20.0"/>
     </joint>
+    <gazebo reference="${prefix}_wheel">
+      <mu1>2.0</mu1>
+      <mu2>2.0</mu2>
+      <kp>1000000.0</kp>
+      <kd>100.0</kd>
+    </gazebo>
   </xacro:macro>
   <xacro:macro name="collector_arm" params="prefix reflect angle limit_lower limit_upper">
@@ -258,3 +264,7 @@
     </plugin>
   </gazebo>
+  <gazebo reference="castor_wheel">
+    <mu1>0.001</mu1>
+    <mu2>0.001</mu2>
+  </gazebo>
 </robot>
