Commit message: WIP: /scan fix attempt

File: ballbot_description/urdf/ballbot.urdf.xacro (robot description, xacro)
@@ -74,5 +74,4 @@
       <origin xyz="0 ${reflect * wheel_y_offset} ${wheel_z_offset}" rpy="0 0 0"/>
       <axis xyz="0 1 0"/>
-      <!-- CRITICAL FIX: Limits are required for Gazebo to apply effort -->
       <limit effort="50.0" velocity="20.0"/>
     </joint>
@@ -134,5 +133,4 @@
     </joint>
   </xacro:macro>
-  <!-- FIX: Added base_footprint to silence KDL warning about root link inertia -->
   <link name="base_footprint"/>
   <joint name="base_joint" type="fixed">
@@ -222,50 +220,5 @@
     <origin xyz="0 0 0.05" rpy="0 0 0"/>
   </joint>
-  <xacro:collector_arm prefix="left" reflect="1" angle="${arm_angle}" limit_lower="-1.57" limit_upper="0.0"/>
-  <xacro:collector_arm prefix="right" reflect="-1" angle="${arm_angle}" limit_lower="0.0" limit_upper="1.57"/>
-  <!-- ROS2 CONTROL -->
-  <ros2_control name="GazeboSimSystem" type="system">
-    <hardware>
-      <plugin>gz_ros2_control/GazeboSimSystem</plugin>
-    </hardware>
-    <!-- Wheels -->
-    <joint name="left_wheel_joint">
-      <command_interface name="velocity">
-        <param name="min">-10</param>
-        <param name="max">10</param>
-      </command_interface>
-      <state_interface name="velocity"/>
-      <state_interface name="position"/>
-    </joint>
-    <joint name="right_wheel_joint">
-      <command_interface name="velocity">
-        <param name="min">-10</param>
-        <param name="max">10</param>
-      </command_interface>
-      <state_interface name="velocity"/>
-      <state_interface name="position"/>
-    </joint>
-    <!-- Flaps -->
-    <joint name="left_flap_joint">
-      <command_interface name="position"/>
-      <state_interface name="position"/>
-      <state_interface name="velocity"/>
-    </joint>
-    <joint name="right_flap_joint">
-      <command_interface name="position"/>
-      <state_interface name="position"/>
-      <state_interface name="velocity"/>
-    </joint>
-  </ros2_control>
-  <!-- Gazebo Plugin for ros2_control -->
-  <gazebo>
-    <plugin filename="gz_ros2_control-system" name="gz_ros2_control::GazeboSimROS2ControlPlugin">
-      <parameters>$(find ballbot_control)/config/ballbot_controllers.yaml</parameters>
-    </plugin>
-  </gazebo>
-  <gazebo reference="castor_wheel">
-    <mu1>0.001</mu1>
-    <mu2>0.001</mu2>
-  </gazebo>
+  <!-- === LIDAR SENSOR PLUGIN START === -->
   <gazebo reference="lidar_link">
     <sensor name="lidar" type="gpu_lidar">
@@ -274,4 +227,6 @@
       <visualize>true</visualize>
       <update_rate>10</update_rate>
+      <topic>scan</topic> <!-- Force topic name to /scan -->
+      <frame_id>lidar_link</frame_id>
       <ray>
         <scan>
@@ -288,8 +243,48 @@
         </range>
       </ray>
-      <plugin filename="gz-sim-sensors-system" name="gz::sim::systems::Sensors">
-        <render_engine>ogre2</render_engine>
-      </plugin>
     </sensor>
   </gazebo>
+  <!-- === LIDAR SENSOR PLUGIN END === -->
+  <xacro:collector_arm prefix="left" reflect="1" angle="${arm_angle}" limit_lower="-1.57" limit_upper="0.0"/>
+  <xacro:collector_arm prefix="right" reflect="-1" angle="${arm_angle}" limit_lower="0.0" limit_upper="1.57"/>
+  <ros2_control name="GazeboSimSystem" type="system">
+    <hardware>
+      <plugin>gz_ros2_control/GazeboSimSystem</plugin>
+    </hardware>
+    <joint name="left_wheel_joint">
+      <command_interface name="velocity">
+        <param name="min">-10</param>
+        <param name="max">10</param>
+      </command_interface>
+      <state_interface name="velocity"/>
+      <state_interface name="position"/>
+    </joint>
+    <joint name="right_wheel_joint">
+      <command_interface name="velocity">
+        <param name="min">-10</param>
+        <param name="max">10</param>
+      </command_interface>
+      <state_interface name="velocity"/>
+      <state_interface name="position"/>
+    </joint>
+    <joint name="left_flap_joint">
+      <command_interface name="position"/>
+      <state_interface name="position"/>
+      <state_interface name="velocity"/>
+    </joint>
+    <joint name="right_flap_joint">
+      <command_interface name="position"/>
+      <state_interface name="position"/>
+      <state_interface name="velocity"/>
+    </joint>
+  </ros2_control>
+  <gazebo>
+    <plugin filename="gz_ros2_control-system" name="gz_ros2_control::GazeboSimROS2ControlPlugin">
+      <parameters>$(find ballbot_control)/config/ballbot_controllers.yaml</parameters>
+    </plugin>
+  </gazebo>
+  <gazebo reference="castor_wheel">
+    <mu1>0.001</mu1>
+    <mu2>0.001</mu2>
+  </gazebo>
 </robot>

Commit message: Update ballbot_description
Adjusted dimensions of the robot to navigate better
Adjusted arm length and positioning to secure the largest obstacle (0.6 dia)
Adjusted flap length to secure smallest obstacle (0.2 dia)

File: ballbot_description/urdf/ballbot.urdf.xacro (robot description, xacro)
@@ -1,23 +1,32 @@
 <?xml version="1.0"?>
 <robot xmlns:xacro="http://www.ros.org/wiki/xacro" name="ballbot">
-  <xacro:property name="chassis_len" value="0.5"/>
-  <xacro:property name="chassis_width" value="0.5"/>
+  <!-- ========================================================================= -->
+  <!-- DIMENSIONS AND PROPERTIES (ADJUSTED) -->
+  <!-- ========================================================================= -->
+  <!-- Chassis (Base) Dimensions -->
+  <xacro:property name="chassis_len" value="0.30"/>   <!-- Length remains 30cm -->
+  <xacro:property name="chassis_width" value="0.65"/> <!-- CHANGED: 0.60 -> 0.65 (Wider by 5cm) -->
   <xacro:property name="chassis_height" value="0.3"/>
   <xacro:property name="chassis_mass" value="3.0"/>
   <xacro:property name="chassis_z_offset" value="0.20"/>
+  <!-- Wheel Dimensions -->
   <xacro:property name="wheel_radius" value="0.05"/>
   <xacro:property name="wheel_width" value="0.04"/>
   <xacro:property name="wheel_mass" value="0.5"/>
-  <xacro:property name="wheel_y_offset" value="0.27"/>
+  <!-- Adjusted wheel separation to fit the new chassis (0.65m width) -->
+  <xacro:property name="wheel_y_offset" value="0.305"/> <!-- ADJUSTED: 0.28 -> 0.305 -->
   <xacro:property name="wheel_z_offset" value="0.05"/>
+  <!-- Castor Dimensions -->
   <xacro:property name="castor_radius" value="0.04"/>
   <xacro:property name="castor_mass" value="1.5"/>
-  <xacro:property name="castor_x_offset" value="-0.2"/>
-  <xacro:property name="arm_len" value="0.6"/>
-  <xacro:property name="arm_width" value="0.05"/>
+  <!-- Castor position remains the same as chassis length is unchanged -->
+  <xacro:property name="castor_x_offset" value="-0.12"/>
+  <!-- Arm and Flap Dimensions -->
+  <xacro:property name="arm_len" value="0.60"/>     <!-- CHANGED: 0.25 -> 0.30 (Longer by 5cm) -->
+  <xacro:property name="arm_width" value="0.03"/>   <!-- Arm width remains 3cm -->
   <xacro:property name="arm_height" value="0.3"/>
   <xacro:property name="arm_mass" value="0.04"/>
-  <xacro:property name="arm_angle" value="0.523"/>
-  <xacro:property name="flap_len" value="0.3"/>
+  <xacro:property name="arm_angle" value="0.0"/>    <!-- Straight forward -->
+  <xacro:property name="flap_len" value="0.25"/>    <!-- CHANGED: 0.19 -> 0.25 (Longer by 6cm) -->
   <xacro:property name="flap_width" value="0.02"/>
   <xacro:property name="flap_height" value="0.3"/>
@@ -28,4 +37,7 @@
   <material name="green"><color rgba="0.0 0.8 0.0 1.0"/></material>
   <material name="red"><color rgba="0.8 0.0 0.0 1.0"/></material>
+  <!-- ========================================================================= -->
+  <!-- MACROS -->
+  <!-- ========================================================================= -->
   <xacro:macro name="box_inertia" params="m x y z">
     <inertial>
@@ -86,4 +98,7 @@
     <link name="${prefix}_arm">
       <visual>
+        <!-- Offset the visual to place the arm's center half its length forward,
+             making the joint origin the base of the arm (x=0) -->
+        <origin xyz="${arm_len/2} 0 0" rpy="0 0 0"/>
         <geometry>
           <box size="${arm_len} ${arm_width} ${arm_height}"/>
@@ -92,4 +107,5 @@
       </visual>
       <collision>
+        <origin xyz="${arm_len/2} 0 0" rpy="0 0 0"/>
         <geometry>
           <box size="${arm_len} ${arm_width} ${arm_height}"/>
@@ -101,5 +117,7 @@
       <parent link="base_link"/>
       <child link="${prefix}_arm"/>
-      <origin xyz="0.51 ${reflect * 0.40} ${chassis_z_offset}" rpy="0 0 ${reflect * angle}"/>
+      <!-- Attach point at the front edge of the chassis (x=chassis_len/2)
+           and set Y position exactly to the chassis edge (chassis_width/2) -->
+      <origin xyz="${chassis_len/2} ${reflect * chassis_width/2} ${chassis_z_offset}" rpy="0 0 ${reflect * angle}"/>
     </joint>
     <link name="${prefix}_flap">
@@ -128,9 +146,13 @@
       <parent link="${prefix}_arm"/>
       <child link="${prefix}_flap"/>
-      <origin xyz="${arm_len/2} 0 0" rpy="0 0 0"/>
+      <!-- Flap joint origin at the end of the arm link (x=arm_len) -->
+      <origin xyz="${arm_len} 0 0" rpy="0 0 0"/>
       <axis xyz="0 0 1"/>
       <limit lower="${limit_lower}" upper="${limit_upper}" effort="10.0" velocity="1.0"/>
     </joint>
   </xacro:macro>
+  <!-- ========================================================================= -->
+  <!-- ROBOT STRUCTURE -->
+  <!-- ========================================================================= -->
   <link name="base_footprint"/>
   <joint name="base_joint" type="fixed">
@@ -247,4 +269,5 @@
   </gazebo>
   <!-- === LIDAR SENSOR PLUGIN END === -->
+  <!-- Arms are now straight (angle=0.0), longer (arm_len=0.30), skinnier (arm_width=0.03), and flaps are 0.22m -->
   <xacro:collector_arm prefix="left" reflect="1" angle="${arm_angle}" limit_lower="-1.57" limit_upper="0.0"/>
   <xacro:collector_arm prefix="right" reflect="-1" angle="${arm_angle}" limit_lower="0.0" limit_upper="1.57"/>

Commit message: Update ballbot_description ballbot_nav2
Major update: Finally implemented nav2 but without colision monitor and IMU integration. Able to publish Nav2 Goal Pose and observe successful path traversal.

File: ballbot_description/urdf/ballbot.urdf.xacro (robot description, xacro)
@@ -6,5 +6,5 @@
   <!-- Chassis (Base) Dimensions -->
   <xacro:property name="chassis_len" value="0.30"/>   <!-- Length remains 30cm -->
-  <xacro:property name="chassis_width" value="0.65"/> <!-- CHANGED: 0.60 -> 0.65 (Wider by 5cm) -->
+  <xacro:property name="chassis_width" value="0.65"/> <!-- Width 65cm -->
   <xacro:property name="chassis_height" value="0.3"/>
   <xacro:property name="chassis_mass" value="3.0"/>
@@ -14,6 +14,6 @@
   <xacro:property name="wheel_width" value="0.04"/>
   <xacro:property name="wheel_mass" value="0.5"/>
-  <!-- Adjusted wheel separation to fit the new chassis (0.65m width) -->
-  <xacro:property name="wheel_y_offset" value="0.305"/> <!-- ADJUSTED: 0.28 -> 0.305 -->
+  <!-- Adjusted wheel separation to fit the chassis (0.65m width) -->
+  <xacro:property name="wheel_y_offset" value="0.305"/>
   <xacro:property name="wheel_z_offset" value="0.05"/>
   <!-- Castor Dimensions -->
@@ -23,10 +23,10 @@
   <xacro:property name="castor_x_offset" value="-0.12"/>
   <!-- Arm and Flap Dimensions -->
-  <xacro:property name="arm_len" value="0.60"/>     <!-- CHANGED: 0.25 -> 0.30 (Longer by 5cm) -->
+  <xacro:property name="arm_len" value="0.60"/>     <!-- User updated: 0.60m -->
   <xacro:property name="arm_width" value="0.03"/>   <!-- Arm width remains 3cm -->
   <xacro:property name="arm_height" value="0.3"/>
   <xacro:property name="arm_mass" value="0.04"/>
   <xacro:property name="arm_angle" value="0.0"/>    <!-- Straight forward -->
-  <xacro:property name="flap_len" value="0.25"/>    <!-- CHANGED: 0.19 -> 0.25 (Longer by 6cm) -->
+  <xacro:property name="flap_len" value="0.25"/>    <!-- User updated: 0.25m -->
   <xacro:property name="flap_width" value="0.02"/>
   <xacro:property name="flap_height" value="0.3"/>
@@ -269,5 +269,5 @@
   </gazebo>
   <!-- === LIDAR SENSOR PLUGIN END === -->
-  <!-- Arms are now straight (angle=0.0), longer (arm_len=0.30), skinnier (arm_width=0.03), and flaps are 0.22m -->
+  <!-- Arms are now straight (angle=0.0), longer (arm_len=0.60), skinnier (arm_width=0.03), and flaps are 0.25m -->
   <xacro:collector_arm prefix="left" reflect="1" angle="${arm_angle}" limit_lower="-1.57" limit_upper="0.0"/>
   <xacro:collector_arm prefix="right" reflect="-1" angle="${arm_angle}" limit_lower="0.0" limit_upper="1.57"/>

Commit message: Created ballbot_imu
Attempted implementation of BNO055 IMU in Ballbot for absolute orientation fusion with odom for accurate mapping and preventing map rotation while navigation.

File: ballbot_description/urdf/ballbot.urdf.xacro (robot description, xacro)
@@ -269,4 +269,95 @@
   </gazebo>
   <!-- === LIDAR SENSOR PLUGIN END === -->
+<!-- === IMU SENSOR PLUGIN START === -->
+<gazebo reference="imu_link">
+  <sensor name="imu_sensor" type="imu">
+    <pose>0 0 0 0 0 0</pose>  <!-- Now relative to imu_link -->
+    <!-- Update rate (BNO055 can do 100Hz) -->
+    <always_on>true</always_on>
+    <update_rate>100</update_rate>
+    <visualize>false</visualize>
+    <!-- Topic name -->
+    <topic>/imu_raw</topic>
+    <!-- IMU sensor configuration -->
+    <imu>
+      <!-- Angular velocity (gyroscope) -->
+      <angular_velocity>
+        <x>
+          <noise type="gaussian">
+            <mean>0.0</mean>
+            <stddev>0.0002</stddev>
+            <bias_mean>0.0000075</bias_mean>
+            <bias_stddev>0.0000008</bias_stddev>
+          </noise>
+        </x>
+        <y>
+          <noise type="gaussian">
+            <mean>0.0</mean>
+            <stddev>0.0002</stddev>
+            <bias_mean>0.0000075</bias_mean>
+            <bias_stddev>0.0000008</bias_stddev>
+          </noise>
+        </y>
+        <z>
+          <noise type="gaussian">
+            <mean>0.0</mean>
+            <stddev>0.0002</stddev>
+            <bias_mean>0.0000075</bias_mean>
+            <bias_stddev>0.0000008</bias_stddev>
+          </noise>
+        </z>
+      </angular_velocity>
+      <!-- Linear acceleration (accelerometer) -->
+      <linear_acceleration>
+        <x>
+          <noise type="gaussian">
+            <mean>0.0</mean>
+            <stddev>0.01</stddev>
+            <bias_mean>0.005</bias_mean>
+            <bias_stddev>0.0002</bias_stddev>
+          </noise>
+        </x>
+        <y>
+          <noise type="gaussian">
+            <mean>0.0</mean>
+            <stddev>0.01</stddev>
+            <bias_mean>0.005</bias_mean>
+            <bias_stddev>0.0002</bias_stddev>
+          </noise>
+        </y>
+        <z>
+          <noise type="gaussian">
+            <mean>0.0</mean>
+            <stddev>0.01</stddev>
+            <bias_mean>0.005</bias_mean>
+            <bias_stddev>0.0002</bias_stddev>
+          </noise>
+        </z>
+      </linear_acceleration>
+    </imu>
+  </sensor>
+</gazebo>
+<!-- Create a separate imu_link for proper TF tree -->
+<link name="imu_link">
+  <visual>
+    <geometry>
+      <box size="0.02 0.02 0.01"/>
+    </geometry>
+    <material name="grey"/>
+  </visual>
+  <collision>
+    <geometry>
+      <box size="0.02 0.02 0.01"/>
+    </geometry>
+  </collision>
+  <xacro:box_inertia m="0.01" x="0.02" y="0.02" z="0.01"/>
+</link>
+<joint name="imu_joint" type="fixed">
+  <parent link="base_link"/>
+  <child link="imu_link"/>
+  <!-- Mount IMU in the center of the chassis -->
+  <origin xyz="0 0 0.2" rpy="0 0 0"/>
+</joint>
+<!-- === IMU SENSOR PLUGIN END === -->
   <!-- Arms are now straight (angle=0.0), longer (arm_len=0.60), skinnier (arm_width=0.03), and flaps are 0.25m -->
   <xacro:collector_arm prefix="left" reflect="1" angle="${arm_angle}" limit_lower="-1.57" limit_upper="0.0"/>
